File: hardware/TinyTX4/TinyTX4-sma.kicad_pcb (KiCad board)
At the start: 2 copper layers, 25 x 47.2 mm, 14 parts, among them J1 Conn_01x03_Male, J2 Conn_01x08_Female, J3 Conn_01x08_Female, J4 Conn_01x08_Female, J5 73391-0060, U1 ATtiny1614-SS, U2 RFM69HW, U3 MCP1703A-3302_SOT23

Commit message: Add printed version
Parts:
- BATT+: renamed from BT1; footprint Connector_Wire:SolderWirePad_1x02_P3.81mm_Drill1mm -> User_Library:SolderWirePad_1x02_P3.81mm_Drill1mm
- J1: footprint Connector_Wire:SolderWirePad_1x03_P3.175mm_Drill1mm -> Connector_PinHeader_2.54mm:PinHeader_1x03_P2.54mm_Vertical
- J5: footprint molex_SMA:MOLEX_73391-0060 -> User_Library:MOLEX_73391-0060
- moved G*** 6.18 mm to (24.4, 54.1)
- moved J1 3.20 mm to (20.6, 58.4), turned to 90 degrees
Connections:
- J3 pad 1: (no net) -> Net-(J3-Pad1)
- J3 pad 2: (no net) -> Net-(J3-Pad2)
- J3 pad 3: (no net) -> Net-(J3-Pad3)
- J3 pad 4: (no net) -> Net-(J3-Pad4)
- J3 pad 5: (no net) -> Net-(J3-Pad5)
- J3 pad 6: (no net) -> Net-(J3-Pad6)
- J3 pad 7: (no net) -> Net-(J3-Pad7)
- J3 pad 8: (no net) -> Net-(J3-Pad8)
- U2 pad 1: (no net) -> Net-(U2-Pad1)
- U2 pad 16: (no net) -> Net-(U2-Pad16)
- U2 pad 3: (no net) -> Net-(U2-Pad3)
- U2 pad 4: (no net) -> Net-(U2-Pad4)
- U2 pad 5: (no net) -> Net-(U2-Pad5)
- U2 pad 6: (no net) -> Net-(U2-Pad6)
- U2 pad 7: (no net) -> Net-(U2-Pad7)
Routing:
- net GND: track 116.5 -> 114.6 mm, vias 13 -> 21
- net Net-(C1-Pad1): track 76.1 -> 78.0 mm
- net Net-(J1-Pad1): track 26.6 -> 27.9 mm
- net Net-(J5-Pad1): track 11.9 -> 13.0 mm
Other:
- board text added: "JLCJLCJLCJLC"
- board text added: "RFM69(H)W"
