File: hardware/TinyTX4/TinyTX4.sch (KiCad schematic (older format))
At the start: 13 parts, among them J1 Conn_01x03_Male, J2 Conn_01x08_Female, J3 Conn_01x08_Female, J4 Conn_01x08_Female, U1 ATtiny1614-SS, U2 RFM69HW, U3 MCP1703A-3302_SOT23

Commit message: Add printed version
Parts:
- added R1, R2: R, symbol Device:R
Connections:
- net GND: now also R2.1
- net at J2.7 (Pin_7), J4.7 (Pin_7): no longer U1.8 (PB1)
- net at J2.8 (Pin_8), J4.8 (Pin_8): no longer U1.9 (PB0)
- net at BT1.1 (+), C3.1, U3.3 (VI): now also R1.2
- new net: R1.1, R2.2, U1.9 (PB0)
Changed lines of the file:
@@
 	1700 3590 1940 3590
 Wire Wire Line
-	1600 4680 1600 3490
-Wire Wire Line
-	1600 3490 1940 3490
-Wire Wire Line
 	1320 3490 1320 3090
 Wire Wire Line
@@
 Wire Wire Line
 	1320 4490 2200 4490
-Wire Wire Line
-	1500 4680 1500 3390
-Wire Wire Line
-	1500 3390 1940 3390
 Connection ~ 2200 4490
 Wire Wire Line
@@
 Wire Wire Line
 	1500 4880 1500 4680
-Connection ~ 1500 4680
 Wire Wire Line
 	1600 4880 1600 4680
-Connection ~ 1600 4680
 Wire Wire Line
 	1700 4880 1700 4680
@@
 Wire Wire Line
 	4430 4490 5270 4490
+$Comp
+L Device:R R1
+U 1 1 605B5BD2
+P 2550 2650
+F 0 "R1" V 2343 2650 50  0000 C CNN
+F 1 "R" V 2434 2650 50  0000 C CNN
+F 2 "" V 2480 2650 50  0001 C CNN
+F 3 "~" H 2550 2650 50  0001 C CNN
+	1    2550 2650
+	0    1    1    0
+$EndComp
+$Comp
+L Device:R R2
+U 1 1 605B6CFB
+P 3000 2650
+F 0 "R2" V 2793 2650 50  0000 C CNN
+F 1 "R" V 2884 2650 50  0000 C CNN
+F 2 "" V 2930 2650 50  0001 C CNN
+F 3 "~" H 3000 2650 50  0001 C CNN
+	1    3000 2650
+	0    1    1    0
+$EndComp
+Wire Wire Line
+	1900 2560 2400 2560
+Wire Wire Line
+	2400 2560 2400 2650
+Connection ~ 1900 2560
+Wire Wire Line
+	2700 2650 2785 2650
+Wire Wire Line
+	3150 2650 3150 2950
+Wire Wire Line
+	3150 2950 1900 2950
+Wire Wire Line
+	1900 2950 1900 2960
+Connection ~ 1900 2960
+Wire Wire Line
+	2785 2650 2785 2800
+Wire Wire Line
+	2785 2800 2305 2800
+Wire Wire Line
+	2305 2800 2305 2910
+Wire Wire Line
+	2305 2910 1985 2910
+Wire Wire Line
+	1985 2910 1985 3230
+Wire Wire Line
+	1985 3230 1915 3230
+Wire Wire Line
+	1915 3230 1915 3390
+Wire Wire Line
+	1915 3390 1940 3390
+Connection ~ 2785 2650
+Wire Wire Line
+	2785 2650 2850 2650
 $EndSCHEMATC
